Commit message: Fixed ur3 wrist orientation

File: ur_description/urdf/ur3.urdf.xacro (robot description, xacro)
@@ -330,5 +330,5 @@
     <link name="${prefix}tool0"/>
     <joint name="${prefix}wrist_3_link-tool0_fixed_joint" type="fixed">
-      <origin xyz="0 ${wrist_3_length} 0" rpy="${pi/-2.0} 0 0"/>
+      <origin xyz="0 ${wrist_3_length} 0" rpy="0 0 ${pi/-2.0}"/>
       <parent link="${prefix}wrist_3_link"/>
       <child link="${prefix}tool0"/>

Commit message: Flipped orientation of wrist on ur3

File: ur_description/urdf/ur3.urdf.xacro (robot description, xacro)
@@ -330,5 +330,5 @@
     <link name="${prefix}tool0"/>
     <joint name="${prefix}wrist_3_link-tool0_fixed_joint" type="fixed">
-      <origin xyz="0 ${wrist_3_length} 0" rpy="0 0 ${pi/-2.0}"/>
+      <origin xyz="0 ${wrist_3_length} 0" rpy="0 0 ${pi/2.0}"/>
       <parent link="${prefix}wrist_3_link"/>
       <child link="${prefix}tool0"/>
